Commit message: update

File: output/test_hand/hand/test_hand.urdf (robot description, URDF)
Before this commit: robot test_hand, 7 links, 6 joints
Links:
- removed link finger2_segment0
- removed link finger2_segment1
Joints:
- removed joint finger2_segment0_joint
- removed joint finger2_segment1_joint
- joint finger0_segment1_joint: origin xyz=0 0 0.5 rpy=0 0 0 -> xyz=0 0 0.6 rpy=0 0 0
- joint finger1_segment0_joint: origin xyz=0.649519052838329 -0.37499999999999983 0 rpy=0 0 1.0471975511965976 -> xyz=9.184850993605148e-17 -0.75 0 rpy=0 0 0.0
- joint finger1_segment1_joint: origin xyz=0 0 0.5 rpy=0 0 0 -> xyz=0 0 0.6 rpy=0 0 0
